File: _autosave-BatteryTelemetry.kicad_pcb (KiCad board)
At the start: 2 copper layers, 55 x 135 mm, 161 parts, among them IC1 BQ76925PWR, IC2 BQ76925PWR, IC3 BQ76925PWR, IC4 BQ76925PWR, J1 Conn_01x07_Pin, J2 Conn_01x07_Pin, J3 Conn_01x07_Pin, J4 Conn_01x07_Pin, J5 USB_C_Receptacle_USB2.0, J6 Conn_01x04_Socket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

Commit message: Layout updated
Routing:
- net +3V3: track 255.1 -> 242.9 mm
- net Net-(U1-GPIO26_ADC0): track 60.8 -> 61.6 mm
Other:
- board text removed: "UART Breakout"
