File: BatteryTelemetry.kicad_pcb (KiCad board)
At the start: 2 copper layers, 55 x 135 mm, 161 parts, among them IC1 BQ76925PWR, IC2 BQ76925PWR, IC3 BQ76925PWR, IC4 BQ76925PWR, J1 Conn_01x07_Pin, J2 Conn_01x07_Pin, J3 Conn_01x07_Pin, J4 Conn_01x07_Pin, J5 USB_C_Receptacle_USB2.0, J6 Conn_01x04_Socket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

Commit message: Logo added
Parts:
- moved R50 2.08 mm to (60.4, 144.0)
- moved R51 2.08 mm to (56.2, 144.0)
Routing:
- net /SDA_BAT4: track 56.8 -> 54.5 mm
- net /SCL_BAT4: track 57.0 -> 54.8 mm
- net +3V3: track 255.1 -> 253.6 mm
- net Net-(U1-GPIO26_ADC0): track 60.8 -> 61.6 mm
Other:
- board text added: "Spring 2024"
- board text added: "TP10"
- board text added: "TP11"
- board text added: "TP12"
- board text added: "TP13"
- board text added: "TP14"
- board text added: "TP15"
- board text added: "TP7"
- board text added: "TP8"
- board text added: "TP9"
